File: Backplane_NT/Backplane_NT.kicad_sch (KiCad schematic)
At the start: 72 parts, among them m12 TestPoint, p12 TestPoint

Commit message: V1.0 release
This release corresponds to V1.0 release of the PCB.
Parts:
- added H1, H2: MountingHole_Pad, MountingHole:MountingHole_2.7mm_M2.5_DIN965_Pad, symbol Mechanical:MountingHole_Pad
- added LAH1, LAH2: MountingHole_Pad, MountingHole:MountingHole_2.2mm_M2_DIN965_Pad, symbol Mechanical:MountingHole_Pad
- added LAM1: LA_Mictor, jdr:LA_Mictor, symbol JDr:LA_Mictor
- added LED1: Conn_01x04_Pin, Connector_PinHeader_2.54mm:PinHeader_1x04_P2.54mm_Vertical, symbol Connector:Conn_01x04_Pin
- added R1, R2: 560, Resistor_THT:R_Axial_DIN0204_L3.6mm_D1.6mm_P7.62mm_Horizontal, symbol Device:R_Small
- added RST1: SW_Push, Button_Switch_THT:SW_PUSH_6mm, symbol Switch:SW_Push
Connections:
- net GND: now also H1.1, H2.1, LAH1.1, LAH2.1, LAM1.1 (nc1), LAM1.3 (GND), LAM1.SH (GND), LED1.4 (Pin_4), RST1.2
- net VCC: now also LED1.1 (Pin_1), R2.2
- net bus0: now also LAM1.37 (d0e)
- net bus1: now also LAM1.35 (d1e)
- net bus10: now also LAM1.17 (d10e)
- net bus11: now also LAM1.15 (d11e)
- net bus12: now also LAM1.13 (d12e)
- net bus13: now also LAM1.11 (d13e)
- net bus14: now also LAM1.9 (d14e)
- net bus15: now also LAM1.7 (d15e)
- net bus2: now also LAM1.33 (d2e)
- net bus3: now also LAM1.31 (d3e)
- net bus4: now also LAM1.29 (d4e)
- net bus5: now also LAM1.27 (d5e)
- net bus6: now also LAM1.25 (d6e)
- net bus7: now also LAM1.23 (d7e)
- net bus8: now also LAM1.21 (d8e)
- net bus9: now also LAM1.19 (d9e)
- net cpu_clk: now also IOB1.BT2, LAM1.5 (clke); no longer IOB1.BH2
- net ioa0: now also IOE1.CU2; no longer IOE1.BE2
- net ioa1: now also IOE1.CT2; no longer IOE1.BF2
- net ioa2: now also IOE1.CS2; no longer IOE1.BF1
- net iod0: now also IOE1.CE1
- net iod1: now also IOE1.CD1
- net iod10: now also IOE1.CM2
- net iod11: now also IOE1.CE2
- net iod12: now also IOE1.CF2
- net iod13: now also IOE1.CH2
- net iod14: now also IOE1.CJ2
- net iod15: now also IOE1.CK2
- net iod2: now also IOE1.CC1
- net iod3: now also IOE1.CB1
- net iod4: now also IOE1.CA1
- net iod5: now also IOE1.CJ1
- net iod6: now also IOE1.CN2
- net iod7: now also IOE1.CH1
- net iod8: now also IOE1.CL2
- net iod9: now also IOE1.CF1
- net mdata6416: now also DSP1.DM2; no longer DSP1.DE2
- net mpi1: now also IOB1.CL1; no longer IOB1.DH2
- net mpo1: now also IOB1.CK1; no longer IOB1.DJ2
- net mpo2: now also IOB1.CP2; no longer IOB1.DL2
- net ms_dt: now also IOB1.AD1; no longer IOB1.AE2
- net pp_rst: now also IOB1.BH2; no longer IOB1.BT2
- net ua0: now also LAM1.38 (d0o)
- net ua1: now also LAM1.36 (d1o)
- net ua10: now also LAM1.18 (d10o)
- net ua11: now also LAM1.16 (d11o)
- net ua2: now also LAM1.34 (d2o)
- net ua3: now also LAM1.32 (d3o)
- net ua4: now also LAM1.30 (d4o)
- net ua5: now also LAM1.28 (d5o)
- net ua6: now also LAM1.26 (d6o)
- net ua7: now also LAM1.24 (d7o)
- net ua8: now also LAM1.22 (d8o)
- net ua9: now also LAM1.20 (d9o)
- net ~{bnk12}: now also IOB1.AE2, IOE1.AE2; no longer IOB1.AD1, IOE1.AD1
- net ~{bnk13}: now also IOB1.AH2, IOE1.AH2; no longer IOB1.AE1, IOE1.AE1
- net ~{bnk14}: now also IOB1.BF1, IOE1.BF1; no longer IOB1.AF1, IOE1.AF1
- net ~{cs1}: no longer IOB1.DE1
- net ~{ds_ioa}: now also IOE1.BA1
- net ~{ds_iod}: now also IOE1.BB1
- net ~{led}: now also IOB1.CR2, R1.2
- net ~{sr_iod}: now also IOE1.BC1
- net xx5: now reaches IOB1.BD1
- net xx5: now also IOE1.BD1
- net ~{sys_rst}: now reaches IOB1.BE1
- net ~{sys_rst}: now also IOE1.BE1, RST1.1
- net xx4: now reaches IOB1.BH1
- net xx4: now also IOE1.BH1
- net dispreq: no longer names the net of DSP1.BT2
- net mpi2: no longer names the net of IOB1.DK2
- net ~{bnk15} renamed xx1
- new net: LED1.3 (Pin_3), R2.1
- new net: LED1.2 (Pin_2), R1.1
- new net xx2: IOB1.AF1, IOE1.AF1
- new net xx3: IOB1.AE1, IOE1.AE1
- no-connect marks 256 -> 232
Other:
- note added: "-Checked-"
- note added: "-Checked/corrected-"
- note added: "-unused-"
- moved on the sheet: C1, C2
