File: DSP_NT/DSP_NT.kicad_pcb (KiCad board)
At the start: 2 copper layers, 233.3 x 152.4 mm, 106 parts, among them J1 Video, J10 Jumper_3_Open, J8 Jumper_3_Open, J9 Jumper_3_Open, U1 74F244, U10 74F374, U11 74F374, U12 74F374, U14 74F166, U15 74F166, U16 74F166, U17 74F166, U18 74F166, U19 74F166, U20 74F166, U21 74F166, U22 74F163, U23 74F163, U24 74F163, U25 74F74, U26 74F00, U29 74F151, U3 74F374, U30 74S02, U32 74F163, U33 74F374, U34 74F374, U35 74F10, U36 74F374, U37 2716, U38 74F163, U39 74F163, U4 74F374, U40 74F374, U42 74F163, U43 74F163, U44 74F244, U45 74F244, U47 74F08, U48 74F74, U49 74F163, U5 74F374, U51 74F00, U52 74F163, U53 74F04, U54 SW_DIP_x08, U55 SW_DIP_x08, U6 74F374, U7 74F374, U8 74F374, U9 74F374, X1 CXO_DIP14, X2 CXO_DIP8

Commit message: V1.0 Release
This release corresponds to V1.0 release of the PCB.
Parts:
- renumbered F1 to MA18, F2 to MA19
Connections:
- DSP1 pad BT2: /dispreq -> unconnected-(DSP1-PadBT2)
Other:
- board text added: "0"
- board text added: "1"
Changed lines of the file:
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@@
 	(net 336 "/vsync")
 	(net 337 "/~{hsync}")
-	(net 338 "/dispreq")
+	(net 338 "unconnected-(DSP1-PadBT2)")
 	(net 339 "/~{vsync}")
 	(net 340 "-12V")
@@
 		)
 		(property "Value" "74F244"
-			(at 3.81 25.19 0)
-			(layer "F.Fab")
+			(at 0.7062 25.19 0)
+			(layer "F.SilkS")
 			(effects
 				(font
@@
 		(descr "Through hole straight pin header, 1x03, 2.54mm pitch, single row")
 		(tags "Through hole pin header THT 1x03 2.54mm single row")
-		(property "Reference" "F1"
-			(at -0.6604 -3.0122 0)
+		(property "Reference" "MA18"
+			(at 1.143 -3.0122 0)
 			(layer "F.SilkS")
 			(effects
@@
 		(descr "Through hole straight pin header, 1x03, 2.54mm pitch, single row")
 		(tags "Through hole pin header THT 1x03 2.54mm single row")
-		(property "Reference" "F2"
+		(property "Reference" "MA19"
 			(at -0.5588 -3.1242 180)
 			(layer "F.SilkS")
@@
 			(keep_end_layers yes)
 			(zone_layer_connections)
-			(net 338 "/dispreq")
+			(net 338 "unconnected-(DSP1-PadBT2)")
 			(pintype "passive+no_connect")
 		)
@@
 		(tags "capacitor handsolder")
 		(property "Reference" "C2"
-			(at 0 -1.85 180)
+			(at 0 -2.54 180)
 			(layer "F.SilkS")
 			(effects
@@
 		(layer "Edge.Cuts")
 	)
+	(gr_text "1"
+		(at 242.4684 116.7384 0)
+		(layer "F.SilkS")
+		(effects
+			(font
+				(size 1 1)
+				(thickness 0.15)
+			)
+		)
+	)
 	(gr_text "Serial:"
 		(at 24.638 168.402 0)
@@
 		)
 	)
-	(gr_text "Field\nselect"
-		(at 245.1862 109.474 0)
+	(gr_text "Field select"
+		(at 241.6556 108.9152 0)
 		(layer "F.SilkS")
 		(effects
@@
 		)
 	)
+	(gr_text "0"
+		(at 242.4176 111.7092 0)
+		(layer "F.SilkS")
+		(effects
+			(font
+				(size 1 1)
+				(thickness 0.15)
+			)
+		)
+	)
