File: DSP_NT/DSP_NT.kicad_sch (KiCad schematic)
At the start: 105 parts, among them J1 Video, J10 Jumper_3_Open, J8 Jumper_3_Open, J9 Jumper_3_Open, U1 74F244, U10 74F374, U11 74F374, U12 74F374, U14 74F166, U15 74F166, U16 74F166, U17 74F166, U18 74F166, U19 74F166, U20 74F166, U21 74F166, U22 74F163, U23 74F163, U24 74F163, U25 74F74, U26 74F00, U29 74F151, U3 74F374, U30 74S02, U32 74F163, U33 74F374, U34 74F374, U35 74F10, U36 74F374, U37 2716, U38 74F163, U39 74F163, U4 74F374, U40 74F374, U42 74F163, U43 74F163, U44 74F244, U45 74F244, U47 74F08, U48 74F74, U49 74F163, U5 74F374, U51 74F00, U52 74F163, U53 74F04, U54 SW_DIP_x08, U55 SW_DIP_x08, U6 74F374, U7 74F374, U8 74F374, U9 74F374, X1 CXO_DIP14, X2 CXO_DIP8

Commit message: V1.0 Release
This release corresponds to V1.0 release of the PCB.
Connections:
- net dispreq: no longer names the net of DSP1.BT2
Changed lines of the file:
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@@
 	)
 	(no_connect
-		(at 40.64 134.62)
+		(at 44.45 134.62)
 	)
 	(no_connect
@@
 	(wire
 		(pts
-			(xy 40.64 134.62) (xy 44.45 134.62)
-		)
-		(stroke
-			(width 0)
-			(type default)
-		)
-	)
-	(wire
-		(pts
 			(xy 74.93 109.22) (xy 82.55 109.22)
 		)
@@
 		)
 	)
-	(label "dispreq"
-		(at 40.64 134.62 180)
-		(effects
-			(font
-				(size 1.27 1.27)
-			)
-			(justify right bottom)
-		)
-	)
