File: IFU_NT/IFU_NT.kicad_pcb (KiCad board)
At the start: 2 copper layers, 233.3 x 152.4 mm, 81 parts, among them U1 74LS283, U10 74LS244, U11 74LS377, U12 74LS244, U13 74LS74, U14 74LS00, U15 74LS04, U16 74LS163, U17 74LS163, U18 74LS163, U19 74LS163, U2 74LS283, U20 74LS138, U21 74LS11, U22 74LS32, U24 74LS374, U25 74S244, U26 74LS374, U27 74LS374, U28 74LS374, U29 74LS374, U3 74LS283, U30 74LS374, U31 74LS374, U32 74LS374, U33 74LS244, U34 74LS163, U35 74LS173, U4 74LS283, U42 74LS374, U5 74LS244, U52 74LS374, U6 74LS244, U7 74LS244, U8 74LS377, U9 74LS244

Commit message: V1.0 Release
This release corresponds to V1.0 release of the PCB.
Parts:
- renumbered F0 to MA17, F1 to MA18, F2 to MA19
Other:
- board text added: "0"
- board text added: "1"
Changed lines of the file:
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@@
 		(descr "Through hole straight pin header, 1x03, 2.54mm pitch, single row")
 		(tags "Through hole pin header THT 1x03 2.54mm single row")
-		(property "Reference" "F0"
+		(property "Reference" "MA17"
 			(at 0 -2.33 0)
 			(layer "F.SilkS")
@@
 		(descr "Through hole straight pin header, 1x03, 2.54mm pitch, single row")
 		(tags "Through hole pin header THT 1x03 2.54mm single row")
-		(property "Reference" "F2"
+		(property "Reference" "MA19"
 			(at 0 -2.33 0)
 			(layer "F.SilkS")
@@
 		(descr "Through hole straight pin header, 1x03, 2.54mm pitch, single row")
 		(tags "Through hole pin header THT 1x03 2.54mm single row")
-		(property "Reference" "F1"
+		(property "Reference" "MA18"
 			(at 0 -2.33 0)
 			(layer "F.SilkS")
@@
 		)
 	)
+	(gr_text "1"
+		(at 140.1572 80.264 0)
+		(layer "F.SilkS")
+		(effects
+			(font
+				(size 1 1)
+				(thickness 0.15)
+			)
+		)
+	)
 	(gr_text "PC + F-> Adr"
 		(at 97.917 83.693 0)
@@
 		)
 	)
+	(gr_text "0"
+		(at 140.4112 75.2856 0)
+		(layer "F.SilkS")
+		(effects
+			(font
+				(size 1 1)
+				(thickness 0.15)
+			)
+		)
+	)
 	(gr_text "Address field"
 		(at 147.193 98.171 0)
@@
 	)
 	(segment
-		(start 211.2772 99.568)
-		(end 211.2772 93.1672)
-		(width 0.3048)
-		(layer "B.Cu")
-		(net 20)
-	)
-	(segment
 		(start 202.4888 120.9548)
 		(end 202.4888 99.6188)
@@
 	(segment
 		(start 211.2772 92.964)
-		(end 211.2772 93.1672)
+		(end 211.2772 99.568)
 		(width 0.3048)
 		(layer "B.Cu")
@@
 	)
 	(segment
-		(start 225.552 93.218)
-		(end 225.557 93.218)
-		(width 0.3048)
-		(layer "F.Cu")
-		(net 26)
-	)
-	(segment
 		(start 224.028 91.694)
 		(end 225.552 93.218)
@@
 	)
 	(segment
-		(start 234.6452 119.38)
-		(end 240.03 119.38)
-		(width 0.3048)
-		(layer "F.Cu")
-		(net 182)
-	)
-	(segment
 		(start 213.233 119.38)
-		(end 234.6452 119.38)
+		(end 240.03 119.38)
 		(width 0.3048)
 		(layer "F.Cu")
