File: IOB_NT/IOB_NT.kicad_pcb (KiCad board)
At the start: 2 copper layers, 233.3 x 152.4 mm, 115 parts, among them J1 Conn_01x03_Pin, J2 Conn_01x03_Pin, J3 Conn_01x03_Pin, J4 Conn_01x04_Pin, U1 Spare, U10 74LS195, U15 LS04, U2 Spare, U21 74LS04, U22 74LS139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

Commit message: V1.0 Release
This release corresponds to V1.0 release of the PCB.
Connections:
- IOB1 pad BF1: unconnected-(IOB1-PadBF1) -> /~{bnk14}
- IODEC1 pad 19: Net-(IODEC1-E1) -> /~{io_dt}
- U21 pad 10: Net-(IODEC1-E1) -> unconnected-(U21-Pad10)
- U21 pad 11: /~{io_dt} -> Net-(U21-Pad11)
- U39 pad 8: unconnected-(U39-Pad8) -> Net-(U21-Pad11)
Routing:
- net /~{bnk14}: track 3.71 -> 137.4 mm, vias 0 -> 7
- net Net-(U21-Pad11): track 0.00 -> 132.5 mm, vias 0 -> 5
- net Net-(IODEC1-E1): track 114.0 -> 0.00 mm, vias 3 -> 0
- net /~{io_dt}: track 122.8 -> 153.4 mm, vias 2 -> 6
- net /bus9: track 66.1 -> 68.5 mm
- net /pp3: track 51.0 -> 49.1 mm, vias 2 -> 1
- net /iod11: track 355.9 -> 354.5 mm
- net /iod4: track 560.7 -> 561.7 mm, vias 20 -> 19
- net /bus14: track 73.0 -> 74.0 mm
- net /iod2: track 579.7 -> 578.7 mm, vias 19 -> 18
- net Net-(PP3-Q0): track 71.4 -> 72.3 mm
- net /~{en_uart1}: track 187.3 -> 188.1 mm
- net Net-(U24-Pad8): track 165.3 -> 166.1 mm
- net /bus12: track 62.5 -> 61.8 mm
- net /~{pps_r}: track 93.9 -> 93.3 mm
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