File: IOB_NT/IOB_NT.kicad_sch (KiCad schematic)
At the start: 114 parts, among them J1 Conn_01x03_Pin, J2 Conn_01x03_Pin, J3 Conn_01x03_Pin, J4 Conn_01x04_Pin, U1 Spare, U10 74LS195, U15 LS04, U2 Spare, U21 74LS04, U22 74LS139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

Commit message: V1.0 Release
This release corresponds to V1.0 release of the PCB.
Connections:
- net ~{bnk14}: now also IOB1.BF1
- net ~{io_dt}: now also IODEC1.19 (E1); no longer U21.11
- net at U39.8: now also U21.11
- net at U21.10: no longer IODEC1.19 (E1)
- no-connect marks 154 -> 153
Other:
- moved on the sheet: U21E, U39C
Changed lines of the file:
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@@
 	)
 	(no_connect
-		(at 72.39 154.94)
-	)
-	(no_connect
 		(at 72.39 152.4)
 	)
@@
 	)
 	(no_connect
-		(at 203.2 374.65)
+		(at 87.63 331.47)
+	)
+	(no_connect
+		(at 53.34 334.01)
 	)
 	(no_connect
@@
 	)
 	(no_connect
-		(at 218.44 372.11)
-	)
-	(no_connect
 		(at 494.03 220.98)
 	)
@@
 	)
 	(no_connect
-		(at 203.2 369.57)
+		(at 53.34 328.93)
 	)
 	(no_connect
@@
 	(wire
 		(pts
-			(xy 71.12 313.69) (xy 74.93 313.69)
+			(xy 82.55 313.69) (xy 92.71 313.69)
 		)
 		(stroke
@@
 	(wire
 		(pts
-			(xy 92.71 313.69) (xy 90.17 313.69)
-		)
-		(stroke
-			(width 0)
-			(type default)
-		)
-	)
-	(wire
-		(pts
 			(xy 554.99 93.98) (xy 557.53 93.98)
 		)
@@
 	(wire
 		(pts
+			(xy 68.58 331.47) (xy 72.39 331.47)
+		)
+		(stroke
+			(width 0)
+			(type default)
+		)
+	)
+	(wire
+		(pts
 			(xy 93.98 48.26) (xy 93.98 54.61)
 		)
@@
 	(wire
 		(pts
+			(xy 72.39 154.94) (xy 80.01 154.94)
+		)
+		(stroke
+			(width 0)
+			(type default)
+		)
+	)
+	(wire
+		(pts
 			(xy 441.96 100.33) (xy 441.96 106.68)
 		)
@@
 	)
 	(label "~{io_dt}"
-		(at 71.12 313.69 180)
+		(at 82.55 313.69 180)
 		(effects
 			(font
@@
 		)
 	)
+	(label "~{bnk14}"
+		(at 80.01 154.94 0)
+		(effects
+			(font
+				(size 1.27 1.27)
+			)
+			(justify left bottom)
+		)
+	)
 	(label "~{fdc}"
 		(at 124.46 289.56 0)
@@
 	(symbol
 		(lib_id "74xx:74LS32")
-		(at 210.82 372.11 0)
+		(at 60.96 331.47 0)
 		(unit 3)
 		(exclude_from_sim no)
@@
 		(dnp no)
 		(property "Reference" "U39"
-			(at 211.074 372.364 0)
+			(at 61.214 331.724 0)
 			(effects
 				(font
@@
 		)
 		(property "Value" "74LS32"
-			(at 216.408 368.554 0)
+			(at 66.548 327.914 0)
 			(effects
 				(font
@@
 		)
 		(property "Footprint" "Package_DIP:DIP-14_W7.62mm"
-			(at 210.82 372.11 0)
+			(at 60.96 331.47 0)
 			(effects
 				(font
@@
 		)
 		(property "Datasheet" "http://www.ti.com/lit/gpn/sn74LS32"
-			(at 210.82 372.11 0)
+			(at 60.96 331.47 0)
 			(effects
 				(font
@@
 		)
 		(property "Description" "Quad 2-input OR"
-			(at 210.82 372.11 0)
+			(at 60.96 331.47 0)
 			(effects
 				(font
@@
 	(symbol
 		(lib_id "74xx:74LS04")
-		(at 82.55 313.69 0)
+		(at 80.01 331.47 0)
 		(unit 5)
 		(exclude_from_sim no)
@@
 		(dnp no)
 		(property "Reference" "U21"
-			(at 81.788 313.436 0)
+			(at 79.248 331.216 0)
 			(effects
 				(font
@@
 		)
 		(property "Value" "74LS04"
-			(at 85.598 310.896 0)
+			(at 83.058 328.676 0)
 			(effects
 				(font
@@
 		)
 		(property "Footprint" "Package_DIP:DIP-14_W7.62mm"
-			(at 82.55 313.69 0)
+			(at 80.01 331.47 0)
 			(effects
 				(font
@@
 		)
 		(property "Datasheet" "http://www.ti.com/lit/gpn/sn74LS04"
-			(at 82.55 313.69 0)
+			(at 80.01 331.47 0)
 			(effects
 				(font
@@
 		)
 		(property "Description" "Hex Inverter"
-			(at 82.55 313.69 0)
+			(at 80.01 331.47 0)
 			(effects
 				(font
